Commit message: Udpated OGm algortihm. We are now subsricbing directly form the gfazebo link topic and then extract the pose. We also defined some physics propertys in our world (cafe) which increased the fps in bgazebo from 30 -> 60 %.

File: src/rvc_simulation_environment/models/robot_vacuum_cleaner/parameter.xacro (robot description, xacro)
@@ -56,5 +56,5 @@
     <xacro:property name="update_rate" value="10"/>
     <xacro:property name="pose_hokuyo_laser_scanner_head" value="0 0 0"/>
-    <xacro:property name="visu_rays" value="true"/>
+    <xacro:property name="visu_rays" value="false"/>
     <xacro:property name="numb_of_samples" value="720"/>
     <xacro:property name="angular_resolution" value="1"/>

Commit message: Adapted friction param and wheel speed param of DDMR.

File: src/rvc_simulation_environment/models/robot_vacuum_cleaner/parameter.xacro (robot description, xacro)
@@ -28,5 +28,5 @@
     <xacro:property name="pos_l_wheel" value="0 0 0"/>                                                                          <!--Origin position of the left wheel -->
     <xacro:property name="pos_r_wheel" value="0 0 0"/>                                                                          <!--Origin position of the right wheel -->
-    <xacro:property name="rot_wheel" value="0.0 1.5707 1.5707"/>                                                                <!--Origin rotation of the wheels -->
+    <xacro:property name="rot_wheel" value="0 ${pi/2} ${pi/2}"/>                                                                <!--Origin rotation of the wheels -->
     <xacro:property name="joint_pos_l_wheel" value="0 ${r_chassis + w_wheel/2} ${h_chassis/2 + dist_chassis_to_ground}"/>       <!--Origin position of the left wheel joint-->
     <xacro:property name="joint_pos_r_wheel" value="0 ${-(r_chassis + w_wheel/2)} ${h_chassis/2 + dist_chassis_to_ground}"/>    <!--Origin position of the right wheel joint-->

File: src/rvc_simulation_environment/models/robot_vacuum_cleaner/robot_vacuum_cleaner.xacro (robot description, xacro)
@@ -36,5 +36,4 @@
         <origin xyz="${pos_chassis}" rpy="${rot_chassis}" />
         <mass value= "${m_chassis}"/>
-        <cylinder_inertia m="${m_chassis}" r="${r_chassis}" h="${h_chassis}"/>
         <xacro:cylinder_inertia m="${m_chassis}" r="${r_chassis}" h="${h_chassis}"/>
     </inertial>
@@ -73,5 +72,4 @@
             <origin xyz="${pos_f_caster_wheel}" rpy="${rot_caster_wheel}"/>
             <mass value= "${m_caster_wheel}"/>
-            <sphere_inertia m="${m_caster_wheel}" r="${r_caster_wheel}"/>
             <xacro:sphere_inertia m="${m_caster_wheel}" r="${r_caster_wheel}"/>
         </inertial>
@@ -110,5 +108,4 @@
             <origin xyz="${pos_b_caster_wheel}" rpy="${rot_caster_wheel}"/>
             <mass value= "${m_caster_wheel}"/>
-            <sphere_inertia m="${m_caster_wheel}" r="${r_caster_wheel}"/>
             <xacro:sphere_inertia m="${m_caster_wheel}" r="${r_caster_wheel}"/>
         </inertial>
@@ -145,5 +142,4 @@
             <origin xyz="${pos_l_wheel}" rpy="${rot_wheel}" />
             <mass value= "${m_wheel}"/>
-            <cylinder_inertia m="${m_wheel}" r="${r_wheel}" h="${w_wheel}"/>
             <xacro:cylinder_inertia m="${m_wheel}" r="${r_wheel}" h="${w_wheel}"/>
         </inertial>
@@ -177,5 +173,4 @@
             <origin xyz="${pos_r_wheel}" rpy="${rot_wheel}" />
             <mass value= "${m_wheel}"/>
-            <cylinder_inertia m="${m_wheel}" r="${r_wheel}" h="${w_wheel}"/>
             <xacro:cylinder_inertia m="${m_wheel}" r="${r_wheel}" h="${w_wheel}"/>
         </inertial>
@@ -188,5 +183,5 @@
         <parent link="base_link"/>
         <limit effort="100" velocity="100"/>
-        <joint_properties damping="0.0" friction="0.0"/>
+        <joint_properties damping="0.2" friction="0.05"/>
     </joint>
     <joint name="base_link_to_right_wheel" type="continuous">
@@ -196,5 +191,5 @@
         <parent link="base_link"/>
         <limit effort="100" velocity="100"/>
-        <joint_properties damping="0.0" friction="0.0"/>
+        <joint_properties damping="0.2" friction="0.05"/>
     </joint>
 <!--____________________________________________________________________________________________________________________________________________________________________-->
@@ -218,5 +213,4 @@
             <origin xyz= "${pos_laser_scanner}" rpy="${rot_laser_scanner}"/>
             <mass value="${m_laser_scanner}"/>
-            <cylinder_inertia m="${m_laser_scanner}" r="${r_laser_scanner}" h="${h_laser_scanner}" />
             <xacro:cylinder_inertia m="${m_laser_scanner}" r="${r_laser_scanner}" h="${h_laser_scanner}" />
         </inertial>

Commit message: Enabled parameter definitions in main launch file and propagate sensor and motion parametrs throuzgh xacro. Also correct an errror that the stddev of the laser hasn't been set to the desired value. Updated playback_node such that motion parameters are automatically red from the ros params into the playback_metadata.json file, when recording data.

File: src/rvc_simulation_environment/models/robot_vacuum_cleaner/parameter.xacro (robot description, xacro)
@@ -63,8 +63,8 @@
     <xacro:property name="min_range" value="0.1"/>                      <!--Minimum distance the lidar can measure-->
     <xacro:property name="max_range" value="10.0"/>                     <!--Maximum distance the lidar can measure-->
-    <xacro:property name="range_resolution" value="0.01"/>
-    <xacro:property name="noise_type" value="gaussian"/>
-    <xacro:property name="noise_mean" value="0.0"/>                     <!--Mean of the gaussian noise in [m]-->
-    <xacro:property name="noise_stddv" value="0.01"/>                   <!--Standard deviation in [m]-->
+    <xacro:property name="range_resolution" value="$(arg laser_range_resolution)"/>
+    <xacro:property name="noise_type" value="$(arg laser_noise_type)"/>
+    <xacro:property name="noise_mean" value="$(arg laser_noise_mean)"/>                     <!--Mean of the gaussian noise in [m]-->
+    <xacro:property name="noise_stddv" value="$(arg laser_noise_stddv)"/>                   <!--Standard deviation in [m]-->
     <xacro:property name="scan_topic" value="/scan"/>
     <xacro:property name="frame_name" value="laser_scanner_link"/>

File: src/rvc_simulation_environment/models/robot_vacuum_cleaner/robot_vacuum_cleaner.xacro (robot description, xacro)
@@ -2,9 +2,13 @@
 <!--Choose a name space and start xacro-->
 <robot name="differential_drive_robot" xmlns:xacro="http://www.ros.org/wiki/xacro">
+    <xacro:arg name="laser_range_resolution" default="0.01"/>
+    <xacro:arg name="laser_noise_type" default="gaussian"/>
+    <xacro:arg name="laser_noise_mean" default="0.0"/>
+    <xacro:arg name="laser_noise_stddv" default="0.01"/>
     <!--Including all xacro files that are needed to describe the robot model-->
-    <xacro:include filename="$(find rvc_simulation_environment)/models/robot_vacuum_cleaner/diff_drive.gazebo"/>
+    <xacro:include filename="$(find rvc_simulation_environment)/models/robot_vacuum_cleaner/parameter.xacro"/>
     <xacro:include filename="$(find rvc_simulation_environment)/models/robot_vacuum_cleaner/materials.xacro"/>
     <xacro:include filename="$(find rvc_simulation_environment)/models/robot_vacuum_cleaner/macros.xacro"/>
-    <xacro:include filename="$(find rvc_simulation_environment)/models/robot_vacuum_cleaner/parameter.xacro"/>
+    <xacro:include filename="$(find rvc_simulation_environment)/models/robot_vacuum_cleaner/diff_drive.gazebo"/>
 <!--____________________________________________________________________________________________________________________________________________________________________-->
 <!--Define Chassis______________________________________________________________________________________________________________________________________________________-->
