Commit message: Added possibility to run robot on the new AWS small indoor map, which represents a realistic indoor apartment. Increase friction parameters in gazebo file cause robot was basically drifting through the new environment before. Now the robot tdrives smoothly through new enviornment. Deleted surface definitions from robot xacro file cause gazeboi file defines all surface parameters of the wheels.

File: src/rvc_simulation_environment/models/robot_vacuum_cleaner/robot_vacuum_cleaner.xacro (robot description, xacro)
@@ -122,39 +122,5 @@
                 <cylinder radius="${r_wheel}" length="${w_wheel}" />
             </geometry>
-            <surface>
-                <!--Reibung-->
-                <friction>
-                    <ode>
-                        <!--Reibungskoeffizienten-->
-                        <mu>1.0</mu>
-                        <mu2>1.0</mu2>
-                        <!--Schlupf-->
-                        <slip1>0.0</slip1>
-                        <slip2>0.0</slip2>
-                    </ode>
-                </friction>
-            </surface>
-        </collision>
-        <visual>
-            <origin xyz="${pos_l_wheel}" rpy="${rot_wheel}" />
-            <geometry>
-                <cylinder radius="${r_wheel}" length="${w_wheel}" />
-            </geometry>
-            <material name="black"/>
-        </visual>
-        <inertial>
-            <origin xyz="${pos_l_wheel}" rpy="${rot_wheel}" />
-            <mass value= "${m_wheel}"/>
-            <xacro:cylinder_inertia m="${m_wheel}" r="${r_wheel}" h="${w_wheel}"/>
-        </inertial>
-    </link>
-    <!--Define the left wheel link of the differential drive mobile robot-->
-    <link name="right_wheel_link">
-        <collision>
-            <origin xyz="${pos_r_wheel}" rpy="${rot_wheel}" />
-            <geometry>
-                <cylinder radius="${r_wheel}" length="${w_wheel}" />
-            </geometry>
-            <surface>
+            <!-- <surface>
                 <friction>
                     <ode>
@@ -165,5 +131,36 @@
                     </ode>
                 </friction>
-            </surface>
+            </surface>                 -->
+        </collision>
+        <visual>
+            <origin xyz="${pos_l_wheel}" rpy="${rot_wheel}" />
+            <geometry>
+                <cylinder radius="${r_wheel}" length="${w_wheel}" />
+            </geometry>
+            <material name="black"/>
+        </visual>
+        <inertial>
+            <origin xyz="${pos_l_wheel}" rpy="${rot_wheel}" />
+            <mass value= "${m_wheel}"/>
+            <xacro:cylinder_inertia m="${m_wheel}" r="${r_wheel}" h="${w_wheel}"/>
+        </inertial>
+    </link>
+    <!--Define the left wheel link of the differential drive mobile robot-->
+    <link name="right_wheel_link">
+        <collision>
+            <origin xyz="${pos_r_wheel}" rpy="${rot_wheel}" />
+            <geometry>
+                <cylinder radius="${r_wheel}" length="${w_wheel}" />
+            </geometry>
+            <!-- <surface>
+                <friction>
+                    <ode>
+                        <mu>1.0</mu>
+                        <mu2>1.0</mu2>
+                        <slip1>0.0</slip1>
+                        <slip2>0.0</slip2>
+                    </ode>
+                </friction>
+            </surface>                 -->
         </collision>
         <visual>
